File: HW3*/KiCad/KiCad.kicad_sch (KiCad schematic)
At the start: 6 parts, among them J1 Power, J2 Digital/PWM, J3 Analog, J4 Digital/PWM

Commit message: fix
Parts:
- added U1: MAX7219, symbol Driver_LED:MAX7219
Connections:
- net *10: now also U1.12 (LOAD)
- net *11: now also U1.1 (DIN)
- net +5V: now also U1.19 (V+)
- net 13: now also U1.13 (CLK)
- net GND: now also U1.4 (GND), U1.9 (GND)
